File: Board/PmodLCD.sch (KiCad schematic (older format))
At the start: 31 parts, among them IC1 FAN533B, P1 PMOD, P2 PMOD, P3 PMOD, P4 PMOD, P5 LCD_BOTTOM, P6 LCD_TOP, P7 TOUCH, SW1 SPST-4

Commit message: Changed Switch Footprint
Parts:
- SW1: footprint Misc:ADF04S04 -> Misc:GDH04S04
Changed lines of the file:
@@
 F 0 "SW1" H 3702 6397 60  0000 R CNN
 F 1 "SPST-4" H 3702 6503 60  0000 R CNN
-F 2 "Misc:ADF04S04" H 3800 6450 60  0001 C CNN
+F 2 "Misc:GDH04S04" H 3800 6450 60  0001 C CNN
 F 3 "" H 3800 6450 60  0000 C CNN
 	1    3800 6450
@@
 F 0 "SW1" H 4202 6397 60  0000 R CNN
 F 1 "SPST-4" H 4202 6503 60  0000 R CNN
-F 2 "Misc:ADF04S04" H 4300 6450 60  0001 C CNN
+F 2 "Misc:GDH04S04" H 4300 6450 60  0001 C CNN
 F 3 "" H 4300 6450 60  0000 C CNN
 	2    4300 6450
@@
 F 0 "SW1" H 4702 6397 60  0000 R CNN
 F 1 "SPST-4" H 4702 6503 60  0000 R CNN
-F 2 "Misc:ADF04S04" H 4800 6450 60  0001 C CNN
+F 2 "Misc:GDH04S04" H 4800 6450 60  0001 C CNN
 F 3 "" H 4800 6450 60  0000 C CNN
 	3    4800 6450
@@
 F 0 "SW1" H 5202 6397 60  0000 R CNN
 F 1 "SPST-4" H 5202 6503 60  0000 R CNN
-F 2 "Misc:ADF04S04" H 5300 6450 60  0001 C CNN
+F 2 "Misc:GDH04S04" H 5300 6450 60  0001 C CNN
 F 3 "" H 5300 6450 60  0000 C CNN
 	4    5300 6450
